File: panel/default_panel/default_panel.kicad_pcb (KiCad board)
At the start: 2 copper layers, 100 x 100 mm, 1 part

Commit message: update board to v1_0_0h
Other:
- board text added: "SOURCE"
- board text added: "default_panel mk_iii for recurBOY v1_0_0 cyberboy666 & ichi raramuri"
- board text removed: "MODE"
- board text removed: "default_panel mk_iii for recurBOY v0_7_1 cyberboy666 & ichi raramuri"
